Commit message: xD

File: catkin_ws/src/zad/model.urdf (robot description, URDF)
Before this commit: robot zad2, 4 links, 3 joints
Links:
- link link2: geometry visual cylinder length=1 radius=0.05
Joints:
- joint joint2: origin xyz=0 0 0.5 rpy=-1.57 0 0 -> xyz=0 0.5 0.5 rpy=-1.57 0 0
- joint joint3: origin xyz=0 0 1 rpy=0 0 0 -> xyz=0 0 0.5 rpy=0 0 0
