Commit message: dziala

File: catkin_ws/src/zad/model2.urdf (robot description, URDF)
Before this commit: robot zad2, 4 links, 3 joints
Links:
- link link2: geometry visual cylinder length=${params['j2']['len']} radius=0.05
- link link3: geometry visual cylinder length=${params['j3']['len']} radius=0.05
Joints:
- joint joint1: origin xyz=0 0 0 rpy=0 0 0 -> xyz=${params['j1']['xyz']} rpy=${params['j1']['rpy']}
- joint joint2: origin xyz=0 0 1 rpy=-1.57 0 0 -> xyz=${params['j2']['xyz']} rpy=${params['j2']['rpy']}
- joint joint3: origin xyz=0 0 1 rpy=0 0 0 -> xyz=${params['j3']['xyz']} rpy=${params['j3']['rpy']}
