Commit message: poprawiony python

File: catkin_ws/src/zad/zad2_model.urdf (robot description, URDF)
Before this commit: robot zad2, 4 links, 3 joints
Links:
- link link1: geometry visual cylinder length=${params['j0']['len']} radius=0.05
- link link2: geometry visual cylinder length=${params['j1']['len']} radius=0.05
- link link3: geometry visual cylinder length=${params['j2']['len']} radius=0.05
Joints:
- joint joint1: axis (none) -> 0 0 1; origin xyz=0 0 0.5 rpy=0 0 0 -> xyz=${params['j0']['xyz']} rpy=${params['j0']['rpy']}
- joint joint2: axis (none) -> 1 0 0; origin xyz=0 0.5 0.5 rpy=-1.57 0 0 -> xyz=${params['j1']['xyz']} rpy=${params['j1']['rpy']}
- joint joint3: axis (none) -> 1 0 0; origin xyz=0 0 0.5 rpy=0 0 0 -> xyz=${params['j2']['xyz']} rpy=${params['j2']['rpy']}

File: catkin_ws/src/zad/zad2_model2.urdf (robot description, URDF)
Before this commit: robot zad2, 4 links, 3 joints
Links:
- link link1: geometry visual cylinder length=${params['j0']['len']} radius=0.05
- link link2: geometry visual cylinder length=${params['j1']['len']} radius=0.05
- link link3: geometry visual cylinder length=${params['j2']['len']} radius=0.05
Joints:
- joint joint1: axis (none) -> 0 0 1; origin xyz=0 0 0.5 rpy=0 0 0 -> xyz=${params['j0']['xyz']} rpy=${params['j0']['rpy']}; type fixed -> continuous
- joint joint2: axis (none) -> 1 0 0; origin xyz=0 0.5 0.5 rpy=-1.57 0 0 -> xyz=${params['j1']['xyz']} rpy=${params['j1']['rpy']}; type fixed -> continuous
- joint joint3: axis (none) -> 1 0 0; origin xyz=0 0 0.5 rpy=0 0 0 -> xyz=${params['j2']['xyz']} rpy=${params['j2']['rpy']}; type fixed -> continuous
