Commit message: nie dziala

File: catkin_ws/src/dh/model.urdf (robot description, URDF)
Before this commit: robot dh, 4 links, 3 joints
Links:
- removed link link4
- added link floor; visual box size=10 10 0
- link link1: geometry visual cylinder length=1 radius=0.2
- link link2: geometry visual cylinder length=1 radius=0.2
- link link3: geometry visual cylinder length=1 radius=0.2
Joints:
- joint joint1: child link2 -> link1; origin xyz=0 0 0 rpy=0 0 0 -> xyz=0 0 0.5 rpy=0 0 0; parent link1 -> floor; type continuous -> fixed
- joint joint2: child link3 -> link2; origin xyz=5 0 0 rpy=-1.57 0 0 -> xyz=0 0 0.5 rpy=-1.57 0 0; parent link2 -> link1; type continuous -> fixed
- joint joint3: child link4 -> link3; origin xyz=5 0 5 rpy=0 0 0 -> xyz=0 0 1 rpy=0 0 0; parent link3 -> link2; type continuous -> fixed
